Commit message: feat: Fix IK/FK coordinate frame pipeline using roboticstoolbox-python standard API
Replace manual TCP offset math with roboticstoolbox-python's standard
robot.tool API (Peter Corke, "Robotics, Vision and Control", 2023).
This fixes TCP showing 0,0,0 at home position and ensures FK/IK use
the same DH model for consistent results.

Key changes:
- IK: Use robot.tool = SE3(tx,ty,tz) instead of manual wp[2]+tcp_z
  offset. ikine_LM automatically accounts for tool via ETS chain.
- FK: Replace COMPAS model.forward_kinematics() (which silently failed)
  with roboticstoolbox DHRobot.fkine() — same model as IK solver.
- Frontend: Pass TCP offset to FK endpoint, check fkResult.valid before
  display, show error when invalid instead of zeros.
- Add coordinate frame labels to all displays (Robot Base Frame,
  Flange Frame, World Frame, Scene).
- UI: Editable home position, joint jog controls, simulation home
  transit, process type sync, deep merge for Zustand persist.
- Remove ungrounded custom code per constitution, replace with
  NotImplementedError stubs citing required library integrations.
- ORNL Slicer 2 integration, milling toolpath, post-processor service.
- 229 tests pass, 0 TypeScript errors.

Co-Authored-By: Claude Opus 4.6 <noreply@anthropic.com>

File: config/urdf/abb_irb6700.urdf (robot description, URDF)
Before this commit: robot abb_irb6700_200_260, 12 links, 11 joints
Links:
- link base_link: geometry collision mesh filename=../meshes/irb6700/collision/base_link.stl; visual mesh filename=../meshes/irb6700/visual/base_link.stl
- link cylinder: geometry collision mesh filename=../meshes/irb6700/collision/cylinder.stl; visual mesh filename=../meshes/irb6700/visual/cylinder.stl
- link link_1: geometry collision mesh filename=../meshes/irb6700/collision/link_1.stl; visual mesh filename=../meshes/irb6700/visual/link_1.stl
- link link_2: geometry collision mesh filename=../meshes/irb6700_200_260/collision/link_2.stl; visual mesh filename=../meshes/irb6700_200_260/visual/link_2.stl
- link link_3: geometry collision mesh filename=../meshes/irb6700_200_260/collision/link_3.stl; visual mesh filename=../meshes/irb6700_200_260/visual/link_3.stl
- link link_4: geometry collision mesh filename=../meshes/irb6700_200_260/collision/link_4.stl; visual mesh filename=../meshes/irb6700_200_260/visual/link_4.stl
- link link_5: geometry collision mesh filename=../meshes/irb6700/collision/link_5.stl; visual mesh filename=../meshes/irb6700/visual/link_5.stl
- link link_6: geometry collision mesh filename=../meshes/irb6700/collision/link_6.stl; visual mesh filename=../meshes/irb6700/visual/link_6.stl
- link piston: geometry collision mesh filename=../meshes/irb6700/collision/piston.stl; visual mesh filename=../meshes/irb6700/visual/piston.stl
